File: PCB/esp32.kicad_sch (KiCad schematic)
At the start: 26 parts, among them IC1 CDCLVC1106PWR, IC2 ESP32-WROOM-32UE-N16, IC3 MMBT3904-AQ, IC4 MMBT3904-AQ

Commit message: Capacitor placement
Moved some decoupling caps from the top to the bottom. Also, file organization
Changed lines of the file:
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@@
 		)
 	)
-	(text_box "ESP32 Programming\nGPIO Pins\n\nInterrupt: 4\nSCLK: 18\nMISO: 19\nMOSI: 23\nReset: 24\n\nEthernet Chip Select:\n5 (Active Low)\n\nStatus LED: 21\n\nLine Decoder\nA0: 25\nA1: 26\nA2: 32\nEnable: 33\n\nUART Clock Frequency:\n14.7456 MHz\n\nSPI speed: <20MHz\n(16 Mhz recommended)\n\nUse Static IP Addressing\n\nUse MQTT (Need a spare\ncomputer)\n\nThermal management is\nhardware triggered. See\npage 7 for more info."
+	(text_box "ESP32 Programming\nGPIO Pins\n\nInterrupt: 4\nSCLK: 18\nMISO: 19\nMOSI: 23\nReset: 24\nOE: 27\n\nEthernet Chip Select:\n5 (Active Low)\n\nStatus LED: 21\n\nLine Decoder\nA0: 25\nA1: 26\nA2: 32\nEnable: 33\n\nUART Clock Frequency:\n14.7456 MHz\n\nSPI speed: <20MHz\n(16 Mhz recommended)\n\nUse Static IP Addressing\n\nUse MQTT (Need a spare\ncomputer)\n\nThermal management is\nhardware triggered. See\npage 7 for more info."
 		(exclude_from_sim no)
 		(at 13.462 13.462 0)
-		(size 23.114 57.6579)
+		(size 23.114 59.1534)
 		(margins 0.9525 0.9525 0.9525 0.9525)
 		(stroke
@@
 	(polyline
 		(pts
-			(xy 14.732 46.228) (xy 33.528 46.228)
-		)
-		(stroke
+			(xy 14.478 47.498) (xy 33.274 47.498)
+		)
+		(stroke

Commit message: Update BOM parts and adjust schematics text/layout
Apply multiple BOM updates and schematic edits: replace/update capacitor, diode, TVS, fuse, regulator, transistor, connector and resistor part numbers and quantities in DarkMagic.csv; add new components (C48/C51/C54, R85-R87, etc.). Change board active layer in DarkMagic.kicad_prl (9 -> 0). Update manufacturer/mouser part numbers for decoupling caps in esp32.kicad_sch and sc16is752_cont..kicad_sch. Tweak sheet text positions/fonts and remove a sentence in sc16is752_cont..kicad_sch, and add a printable installer-sign text block to sensor_pinout.kicad_sch for cable verification. These edits reflect revised part selections and improve schematic documentation/readability.
Parts:
- C3, C4: Manufacturer_Part_Number CL21A106KAYNNNF -> CL21A106KBYQNNE; Mouser Part Number 187-CL21A106KAYNNNF -> 187-CL21A106KBYQNNE
Changed lines of the file:
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@@
 			)
 		)
-		(property "Manufacturer_Part_Number" "CL21A106KAYNNNF "
+		(property "Manufacturer_Part_Number" "CL21A106KBYQNNE"
 			(at 49.53 49.53 0)
 			(hide yes)
@@
 			)
 		)
-		(property "Mouser Part Number" "187-CL21A106KAYNNNF "
+		(property "Mouser Part Number" "187-CL21A106KBYQNNE "
 			(at 49.53 49.53 0)
 			(hide yes)
@@
 			)
 		)
-		(property "Manufacturer_Part_Number" "CL21A106KAYNNNF "
+		(property "Manufacturer_Part_Number" "CL21A106KBYQNNE"
 			(at 62.23 26.67 0)
 			(hide yes)
@@
 			)
 		)
-		(property "Mouser Part Number" "187-CL21A106KAYNNNF "
+		(property "Mouser Part Number" "187-CL21A106KBYQNNE "
 			(at 62.23 26.67 0)
 			(hide yes)
