File: PCB/esp32.kicad_sch (KiCad schematic)
At the start: 26 parts, among them IC1 CDCLVC1106PWR, IC2 ESP32-WROOM-32UE-N16, IC3 MMBT3904-AQ, IC4 MMBT3904-AQ

Commit message: Add 1x04 pin socket and clean footprint attrs
Inserted a new 1x04 vertical pin socket footprint (J9) for the ESP32 connector and added corresponding silk labels for IO pins. Removed stray "dnp" attributes from multiple footprint pad definitions (smd/through_hole) to enable those pads, added units/pin listings for a couple hierarchical sheet refs, and adjusted several silkscreen/text positions and rotations (IC1, R4, C3, L1, TEA@CPP text). Also includes minor polygon/coordinate updates and other small layout cleanups in PCB/DarkMagic.kicad_pcb.
Parts:
- added J9: Conn_01x04, Connector_PinSocket_2.54mm:PinSocket_1x04_P2.54mm_Vertical, symbol Connector_Generic:Conn_01x04
- V1: now not fitted
Connections:
- net IO13: now also J9.3 (Pin_3)
- net IO14: now also J9.4 (Pin_4)
- net IO16: now also J9.2 (Pin_2)
- net IO17: now also J9.1 (Pin_1)
Changed lines of the file:
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@@
 		)
 	)
+	(wire
+		(pts
+			(xy 128.27 64.77) (xy 128.27 68.58)
+		)
+		(stroke
+			(width 0)
+			(type default)
+		)
+	)
 	(polyline
 		(pts
@@
 		)
 	)
+	(wire
+		(pts
+			(xy 123.19 64.77) (xy 123.19 68.58)
+		)
+		(stroke
+			(width 0)
+			(type default)
+		)
+	)
 	(polyline
 		(pts
@@
 		)
 	)
+	(wire
+		(pts
+			(xy 130.81 64.77) (xy 130.81 68.58)
+		)
+		(stroke
+			(width 0)
+			(type default)
+		)
+	)
 	(polyline
 		(pts
@@
 		)
 	)
+	(wire
+		(pts
+			(xy 125.73 64.77) (xy 125.73 68.58)
+		)
+		(stroke
+			(width 0)
+			(type default)
+		)
+	)
 	(polyline
 		(pts
@@
 		)
 	)
+	(label "IO14"
+		(at 123.19 64.77 270)
+		(effects
+			(font
+				(size 1.27 1.27)
+			)
+			(justify right bottom)
+		)
+	)
 	(label "GND"
 		(at 27.432 151.13 0)
@@
 		)
 	)
+	(label "IO17"
+		(at 130.81 64.77 270)
+		(effects
+			(font
+				(size 1.27 1.27)
+			)
+			(justify right bottom)
+		)
+	)
 	(label "XTAL"
 		(at 27.432 135.89 0)
@@
 		)
 	)
+	(label "IO13"
+		(at 125.73 64.77 270)
+		(effects
+			(font
+				(size 1.27 1.27)
+			)
+			(justify right bottom)
+		)
+	)
 	(label "IO21"
 		(at 125.73 49.53 180)
@@
 		)
 	)
+	(label "IO16"
+		(at 128.27 64.77 270)
+		(effects
+			(font
+				(size 1.27 1.27)
+			)
+			(justify right bottom)
+		)
+	)
 	(label "GND"
 		(at 27.432 138.43 0)
@@
 		(on_board yes)
 		(in_pos_files yes)
-		(dnp no)
+		(dnp yes)
 		(property "Reference" "V1"
 			(at 22.7302 180.34 0)
@@
 					(unit 1)
 				)
+			)
+		)
+	)
+	(symbol
+		(lib_id "Connector_Generic:Conn_01x04")
+		(at 128.27 73.66 270)
+		(unit 1)
+		(body_style 1)
+		(exclude_from_sim no)
+		(in_bom no)
+		(on_board yes)
+		(in_pos_files yes)
+		(dnp no)
+		(property "Reference" "J9"
+			(at 120.904 76.708 90)
+			(show_name no)
+			(do_not_autoplace no)
+			(effects
+				(font
+					(size 1.27 1.27)
+				)
+				(justify left)
+			)
+		)
+		(property "Value" "Conn_01x04"
+			(at 120.904 79.248 90)
+			(show_name no)
+			(do_not_autoplace no)
+			(effects
+				(font
+					(size 1.27 1.27)
+				)
+				(justify left)
+			)
+		)
+		(property "Footprint" "Connector_PinSocket_2.54mm:PinSocket_1x04_P2.54mm_Vertical"
+			(at 128.27 73.66 0)
+			(hide yes)
+			(show_name no)
+			(do_not_autoplace no)
+			(effects
+				(font
+					(size 1.27 1.27)
+				)
+			)
+		)
+		(property "Datasheet" ""
+			(at 128.27 73.66 0)
+			(hide yes)
+			(show_name no)
+			(do_not_autoplace no)
+			(effects
+				(font
+					(size 1.27 1.27)
+				)
+			)
+		)
+		(property "Description" "Generic connector, single row, 01x04, script generated (kicad-library-utils/schlib/autogen/connector/)"
+			(at 128.27 73.66 0)
+			(hide yes)
+			(show_name no)
+			(do_not_autoplace no)
+			(effects
+				(font
+					(size 1.27 1.27)
+				)
+			)
+		)
+		(pin "3"
+		)
+		(pin "1"
+		)
+		(pin "2"
+		)
+		(pin "4"
+		)
+		(instances
+			(project "DarkMagic"
+				(path "/8bdb7bb0-7fad-47bb-9a1b-904625b99d57"
+					(reference "J9")
+					(unit 1)
+				)

Commit message: Add bottom hand-solder caps and update BOM
Update PCB to add bottom-side hand-solder 0805 capacitor footprints and sync BOM. DarkMagic.csv: increment 0.1uF part count (34→35) and 4.7uF count (1→2) and update component lists. DarkMagic.kicad_pcb: add two B.Cu hand-solder capacitor footprints (C7, C10), adjust several footprint attributes (mark many SMD/TH pads as DNP or set solder_mask_margin), tweak some pad/part positions and UUIDs, and rename one net from /USB_VBUS to /CP_VBUS. Also add generated files (PCB/bom/ibom.html and PCB/database/project.db) and other production file updates to keep project metadata in sync.
Parts:
- V1: now fitted
Changed lines of the file:
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@@
 		(on_board yes)
 		(in_pos_files yes)
-		(dnp yes)
+		(dnp no)
 		(property "Reference" "V1"
 			(at 22.7302 180.34 0)

Commit message: PCB: Reroute nets and update component value
Modify DarkMagic.kicad_pcb to correct power routing and update a component value. Changes include: changed a component Value from "CDCLVC1106PWR" to "5PB1106PGGI8", reassigned a pad/net from GND to +3V3, moved a via, removed and added several F.Cu segments (cleaned up GND segments and added +3V3 traces), and adjusted a board polygon/outline coordinate. These edits fix net connections and reflect the correct part designation in the PCB layout.
Parts:
- IC1: value CDCLVC1106PWR -> 5PB1106PGGI8; Manufacturer_Name Texas Instruments -> Renesas Electronics; Manufacturer_Part_Number CDCLVC1106PWR -> 5PB1106PGGI8; Maunfacturer Part Number (none) -> 5PB1106PGGI8; Maunfacturer_Part_Number (none) -> 972-5PB1106PGGI8; Mouser Part Number 595-CDCLVC1106PWR -> 972-5PB1106PGGI8; Mouser Price/Stock https://www.mouser.co.uk/ProductDetail/Texas-Instruments/CD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 -> https://www.mouser.com/ProductDetail/Renesas-Electronics/5P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
Connections:
- net +3V3: now also IC1.2 (1G)
- net GND: no longer IC1.2 (1G)
Changed lines of the file:
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@@
 	)
 	(junction
+		(at 20.32 138.43)
+		(diameter 0)
+		(color 0 0 0 0)
+	)
+	(junction
 		(at 118.11 85.09)
 		(diameter 0)
@@
 	)
 	(junction
-		(at 22.352 146.05)
-		(diameter 0)
-		(color 0 0 0 0)
-	)
-	(junction
 		(at 118.11 67.31)
 		(diameter 0)
@@
 	)
 	(junction
+		(at 20.32 146.05)
+		(diameter 0)
+		(color 0 0 0 0)
+	)
+	(junction
 		(at 49.53 64.77)
 		(diameter 0)
@@
 	(wire
 		(pts
-			(xy 19.812 146.05) (xy 19.812 143.51)
+			(xy 20.32 146.05) (xy 20.32 138.43)
 		)
 		(stroke
@@
 		)
 	)
-	(wire
-		(pts
-			(xy 22.352 146.05) (xy 36.322 146.05)
-		)
-		(stroke
-			(width 0)
-			(type default)
-		)
-	)
 	(polyline
 		(pts
@@
 	(wire
 		(pts
-			(xy 22.352 146.05) (xy 22.352 148.59)
+			(xy 20.32 146.05) (xy 20.32 148.59)
 		)
 		(stroke
@@
 	(wire
 		(pts
-			(xy 22.352 157.48) (xy 27.432 157.48)
+			(xy 20.32 157.48) (xy 27.432 157.48)
 		)
 		(stroke
@@
 		)
 	)
+	(wire
+		(pts
+			(xy 20.32 138.43) (xy 20.32 135.89)
+		)
+		(stroke
+			(width 0)
+			(type default)
+		)
+	)
 	(polyline
 		(pts
@@
 	(wire
 		(pts
-			(xy 22.352 156.21) (xy 22.352 157.48)
+			(xy 20.32 156.21) (xy 20.32 157.48)
 		)
 		(stroke
@@
 	(wire
 		(pts
-			(xy 27.432 138.43) (xy 36.322 138.43)
+			(xy 20.32 138.43) (xy 36.322 138.43)
 		)
 		(stroke
@@
 	(wire
 		(pts
-			(xy 19.812 146.05) (xy 22.352 146.05)
+			(xy 20.32 146.05) (xy 36.322 146.05)
 		)
 		(stroke
@@
 		)
 	)
-	(label "GND"
-		(at 27.432 138.43 0)
-		(effects
-			(font
-				(size 1.27 1.27)
-			)
-			(justify left bottom)
-		)
-	)
 	(label "IO14"
 		(at 63.5 59.69 0)
@@
 	(symbol
 		(lib_id "Device:C")
-		(at 22.352 152.4 180)
+		(at 20.32 152.4 180)
 		(unit 1)
 		(body_style 1)
@@
 		(dnp no)
 		(property "Reference" "C1"
-			(at 16.256 152.4 0)
+			(at 14.224 152.4 0)
 			(show_name no)
 			(do_not_autoplace no)
@@
 		)
 		(property "Value" "0.1uF"
-			(at 16.002 154.94 0)
+			(at 13.97 154.94 0)
 			(show_name no)
 			(do_not_autoplace no)
@@
 		)
 		(property "Footprint" "Capacitor_SMD:C_0805_2012Metric_Pad1.18x1.45mm_HandSolder"
-			(at 21.3868 148.59 0)
+			(at 19.3548 148.59 0)
 			(hide yes)
 			(show_name no)
@@
 		)
 		(property "Datasheet" ""
-			(at 22.352 152.4 0)
+			(at 20.32 152.4 0)
 			(hide yes)
 			(show_name no)
@@
 		)
 		(property "Description" "Unpolarized capacitor"
-			(at 22.352 152.4 0)
+			(at 20.32 152.4 0)
 			(hide yes)
 			(show_name no)
@@
 		)
 		(property "Manufacturer_Part_Number" "CL21B104KCC5PNC "
-			(at 22.352 152.4 0)
+			(at 20.32 152.4 0)
 			(hide yes)
 			(show_name no)
@@
 		)
 		(property "Mouser Part Number" "187-CL21B104KCC5PNC "
-			(at 22.352 152.4 0)
+			(at 20.32 152.4 0)
 			(hide yes)
 			(show_name no)
@@
 		)
 		(property "Maunfacturer Part Number" ""
-			(at 22.352 152.4 0)
+			(at 20.32 152.4 0)
 			(hide yes)
 			(show_name no)
@@
 		)
 		(property "AVAILABILITY" ""
-			(at 22.352 152.4 0)
+			(at 20.32 152.4 0)
 			(hide yes)
 			(show_name no)
@@
 		)
 		(property "Check_prices" ""
-			(at 22.352 152.4 0)
+			(at 20.32 152.4 0)
 			(hide yes)
 			(show_name no)
@@
 		)
 		(property "MF" ""
-			(at 22.352 152.4 0)
+			(at 20.32 152.4 0)
 			(hide yes)
 			(show_name no)
@@
 		)
 		(property "MP" ""
-			(at 22.352 152.4 0)
+			(at 20.32 152.4 0)
 			(hide yes)
 			(show_name no)
@@
 		)
 		(property "Maunfacturer_Part_Number" ""
-			(at 22.352 152.4 0)
+			(at 20.32 152.4 0)
 			(hide yes)
 			(show_name no)
@@
 		)
 		(property "PACKAGE" ""
-			(at 22.352 152.4 0)
+			(at 20.32 152.4 0)
 			(hide yes)
 			(show_name no)
@@
 		)
 		(property "PARTREV" ""
-			(at 22.352 152.4 0)
+			(at 20.32 152.4 0)
 			(hide yes)
 			(show_name no)
@@
 		)
 		(property "PRICE" ""
-			(at 22.352 152.4 0)
+			(at 20.32 152.4 0)
 			(hide yes)
 			(show_name no)
@@
 		)
 		(property "STANDARD" ""
-			(at 22.352 152.4 0)
+			(at 20.32 152.4 0)
 			(hide yes)
 			(show_name no)
@@
 		)
 		(property "SnapEDA_Link" ""
-			(at 22.352 152.4 0)
+			(at 20.32 152.4 0)
 			(hide yes)
 			(show_name no)
@@
 			)
 		)
-		(property "Value" "CDCLVC1106PWR"
+		(property "Value" "5PB1106PGGI8"
 			(at 51.562 130.81 0)
 			(show_name no)
@@
 			)
 		)
-		(property "Datasheet" "http://www.ti.com/lit/ds/symlink/cdclvc1108.pdf"
+		(property "Datasheet" "https://www.renesas.com/en/document/dst/5pb11xx-family-datasheet"
 			(at 62.992 330.81 0)
 			(hide yes)
@@
 			)
 		)
-		(property "Mouser Part Number" "595-CDCLVC1106PWR"
+		(property "Mouser Part Number" "972-5PB1106PGGI8 "
 			(at 62.992 630.81 0)
 			(hide yes)
@@
 			)
 		)
-		(property "Mouser Price/Stock" "https://www.mouser.co.uk/ProductDetail/Texas-Instruments/CDCLVC1106PWR?qs=CLImetaeaXVZfWEl0J7gng%3D%3D"
+		(property "Mouser Price/Stock" "https://www.mouser.com/ProductDetail/Renesas-Electronics/5PB1106PGGI8?qs=3FEoAYHLzoCwnPaY3KQFFw%3D%3D"
 			(at 62.992 730.81 0)
 			(hide yes)
@@
 			)
 		)
-		(property "Manufacturer_Name" "Texas Instruments"
+		(property "Manufacturer_Name" "Renesas Electronics"
 			(at 62.992 830.81 0)
 			(hide yes)
@@
 			)
 		)
-		(property "Manufacturer_Part_Number" "CDCLVC1106PWR"
+		(property "Manufacturer_Part_Number" "5PB1106PGGI8 "
 			(at 62.992 930.81 0)
 			(hide yes)
@@
 			)
 		)
-		(property "Maunfacturer Part Number" ""
+		(property "Maunfacturer Part Number" "5PB1106PGGI8 "
 			(at 36.322 135.89 0)
 			(hide yes)
@@
 			)
 		)
-		(property "Maunfacturer_Part_Number" ""
+		(property "Maunfacturer_Part_Number" "972-5PB1106PGGI8 "
 			(at 36.322 135.89 0)
 			(hide yes)
@@
 	(symbol
 		(lib_id "power:+3V3")
-		(at 19.812 143.51 0)
+		(at 20.32 135.89 0)
 		(unit 1)
 		(body_style 1)
@@
 		(fields_autoplaced yes)
 		(property "Reference" "#PWR01"
-			(at 19.812 147.32 0)
+			(at 20.32 139.7 0)
 			(hide yes)
 			(show_name no)
@@
 		)
 		(property "Value" "+3V3"
-			(at 19.812 138.43 0)
+			(at 20.32 130.81 0)
 			(show_name no)
 			(do_not_autoplace no)
@@
 		)
 		(property "Footprint" ""
-			(at 19.812 143.51 0)
+			(at 20.32 135.89 0)
 			(hide yes)
 			(show_name no)
@@
 		)
 		(property "Datasheet" ""
-			(at 19.812 143.51 0)
+			(at 20.32 135.89 0)
 			(hide yes)
 			(show_name no)
@@
 		)
 		(property "Description" "Power symbol creates a global label with name \"+3V3\""
-			(at 19.812 143.51 0)
+			(at 20.32 135.89 0)
 			(hide yes)
 			(show_name no)

Commit message: Add 0805 handsolder footprint and reroute nets
Add an 0805 hand-solder capacitor footprint (Pad1.18x1.45mm) on B.Cu (C50) and update existing 0805 footprint reference placement. Add copper segments and a via to connect +3V3 and GND between F.Cu and B.Cu (including new via at 148.675,37.84). Re-route several F.Cu traces (ESP_A1 and +3V3) and update segment coordinates/UUIDs. Adjust a copper zone (changed layer to F.Mask and lowered priority) and remove/replace some filled polygons. Update associated project/schematic metadata files and add schematic lock file.
Changed lines of the file:
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@@
 	(wire
 		(pts
-			(xy 16.51 186.69) (xy 16.51 190.5)
+			(xy 16.51 186.69) (xy 16.51 194.31)
 		)
 		(stroke
@@
 	(wire
 		(pts
-			(xy 16.51 175.26) (xy 16.51 176.53)
+			(xy 16.51 172.72) (xy 16.51 176.53)
 		)
 		(stroke
@@
 	(wire
 		(pts
-			(xy 16.51 190.5) (xy 17.78 190.5)
+			(xy 16.51 194.31) (xy 17.78 194.31)
 		)
 		(stroke
@@
 	(symbol
 		(lib_id "power:+12V")
-		(at 16.51 175.26 0)
+		(at 16.51 172.72 0)
 		(unit 1)
 		(body_style 1)
@@
 		(dnp no)
 		(property "Reference" "#PWR095"
-			(at 16.51 179.07 0)
+			(at 16.51 176.53 0)
 			(hide yes)
 			(show_name no)
@@
 		)
 		(property "Value" "+12V"
-			(at 13.462 171.196 0)
+			(at 13.462 168.656 0)
 			(show_name no)
 			(do_not_autoplace no)
@@
 		)
 		(property "Footprint" ""
-			(at 16.51 175.26 0)
+			(at 16.51 172.72 0)
 			(hide yes)
 			(show_name no)
@@
 		)
 		(property "Datasheet" ""
-			(at 16.51 175.26 0)
+			(at 16.51 172.72 0)
 			(hide yes)
 			(show_name no)
@@
 		)
 		(property "Description" "Power symbol creates a global label with name \"+12V\""
-			(at 16.51 175.26 0)
+			(at 16.51 172.72 0)
 			(hide yes)
 			(show_name no)
@@
 	(symbol
 		(lib_id "power:GND")
-		(at 17.78 190.5 90)
+		(at 17.78 194.31 90)
 		(unit 1)
 		(body_style 1)
@@
 		(dnp no)
 		(property "Reference" "#PWR096"
-			(at 24.13 190.5 0)
+			(at 24.13 194.31 0)
 			(hide yes)
 			(show_name no)
@@
 		)
 		(property "Value" "GND"
-			(at 21.082 190.5 90)
+			(at 21.082 194.31 90)
 			(show_name no)
 			(do_not_autoplace no)
@@
 		)
 		(property "Footprint" ""
-			(at 17.78 190.5 0)
+			(at 17.78 194.31 0)
 			(hide yes)
 			(show_name no)
@@
 		)
 		(property "Datasheet" ""
-			(at 17.78 190.5 0)
+			(at 17.78 194.31 0)
 			(hide yes)
 			(show_name no)
@@
 		)
 		(property "Description" "Power symbol creates a global label with name \"GND\" , ground"
-			(at 17.78 190.5 0)
+			(at 17.78 194.31 0)
 			(hide yes)
 			(show_name no)
