File: PCB/esp32.kicad_sch (KiCad schematic)
At the start: 27 parts, among them IC1 5PB1106PGGI8, IC2 ESP32-WROOM-32UE-N16, IC3 MMBT3904-AQ, IC4 MMBT3904-AQ, J9 Conn_01x04

Commit message: feat: initialize project with ESP32 schematic, ethernet port layout, and base firmware.
Changed lines of the file:
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@@
 		)
 	)
-	(text_box "ESP32 Programming\nGPIO Pins\n\nInterrupt: 4\nSCLK: 18\nMISO: 19\nMOSI: 23\nReset: 24\nOE: 27\n\nEthernet Chip Select:\n5 (Active Low)\n\nStatus LED: 21\n\nLine Decoder\nA0: 25\nA1: 26\nA2: 32\nEnable: 33\n\nUART Clock Frequency:\n14.7456 MHz\n\nSPI speed: <20MHz\n(16 Mhz recommended)\n\nUse Static IP Addressing\n\nUse MQTT (Need a spare\ncomputer)\n\nThermal management is\nhardware triggered. See\npage 7 for more info."
+	(text_box "ESP32 Programming\nGPIO Pins\n\nInterrupt: 4\nSCLK: 18\nMISO: 19\nMOSI: 23\nReset: 2\nOE: 27\n\nEthernet Chip Select:\n5 (Active Low)\n\nStatus LED: 21\n\nLine Decoder\nA0: 25\nA1: 26\nA2: 32\nEnable: 33\n\nUART Clock Frequency:\n14.7456 MHz\n\nSPI speed: <20MHz\n(16 Mhz recommended)\n\nUse Static IP Addressing\n\nUse MQTT (Need a spare\ncomputer)\n\nThermal management is\nhardware triggered. See\npage 7 for more info."
 		(exclude_from_sim no)
 		(at 13.462 13.462 0)
