File: PCB/esp32.kicad_sch (KiCad schematic)
At the start: 27 parts, among them IC1 5PB1106PGGI8, IC2 ESP32-WROOM-32UE-N16, IC3 MMBT3904-AQ, IC4 MMBT3904-AQ, J9 Conn_01x04

Commit message: Board Modifications and Initial Comms w/ Sensors
Modified wiring to separate ethernet reset from SC16 reset, adjusted pinouts and power, worked on code to get board talking to sensors. Ethernet still needs a bodge wire at this point.
Connections:
- net +3V3: now also J9.4 (Pin_4)
- net ESP_USRSTT: now also IC2.13 (IO14); no longer IC2.24 (IO2)
- net GND: now also J9.3 (Pin_3)
- net IO13 renamed W5500_RST
- net W5500_RST: no longer J9.3 (Pin_3)
- removed net IO14: IC2.13 (IO14), J9.4 (Pin_4)

Commit message: Diagnosing Ethernet Controller
The Ethernet chip is dead, we'll need a new one. Minor optimizations everywhere.
Connections:
- net +3V3: now also J9.3 (Pin_3); no longer J9.4 (Pin_4)
- net GND: now also J9.4 (Pin_4); no longer J9.3 (Pin_3)
- net IO15: no longer names the net of IC2.23 (IO15)
- no-connect marks 9 -> 11
Changed lines of the file:
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@@
 		)
 	)
-	(text_box "ESP32 Programming\nGPIO Pins\n\nInterrupt: 4\nSCLK: 18\nMISO: 19\nMOSI: 23\nReset: 2\nOE: 27\n\nEthernet Chip Select:\n5 (Active Low)\nETH Reset: 13\n\nStatus LED: 21\n\nLine Decoder\nA0: 25\nA1: 26\nA2: 32\nEnable: 33\n\nUART Clock Frequency:\n14.7456 MHz\n\nSPI speed: <20MHz\n(16 Mhz recommended)\n\nUse Static IP Addressing\n\nUse MQTT (Need a spare\ncomputer)\n\nThermal management is\nhardware triggered. See\npage 7 for more info."
+	(text_box "ESP32 Programming\nGPIO Pins\n\nInterrupt: 4\nSCLK: 18\nMISO: 19\nMOSI: 23\nReset: 2\nOE: 27\n\nEthernet Chip Select:\n5 (Active Low)\nETH Reset: 13\n\nStatus LED: 21\n\nLine Decoder\nA0: 25\nA1: 26\nA2: 32\nEnable: 33\n\nSpare IO Pins: 16, 17\n\nUART Clock Frequency:\n14.7456 MHz\n\nSPI speed: <20MHz\n(16 Mhz recommended)\n\nUse Static IP Addressing\n\nUse MQTT (Need a spare\ncomputer)\n\nThermal management is\nhardware triggered. See\npage 7 for more info."
 		(exclude_from_sim no)
 		(at 13.462 13.462 0)
-		(size 23.114 61.468)
+		(size 23.114 64.0605)
 		(margins 0.9525 0.9525 0.9525 0.9525)
 		(stroke
@@
 	)
 	(no_connect
+		(at 76.2 87.63)
+	)
+	(no_connect
 		(at 76.2 39.37)
 	)
@@
 	)
 	(no_connect
+		(at 76.2 85.09)
+	)
+	(no_connect
 		(at 76.2 82.55)
 	)
@@
 	(polyline
 		(pts
-			(xy 14.605 48.895) (xy 33.401 48.895)
+			(xy 14.605 52.07) (xy 33.401 52.07)
 		)
 		(stroke
@@
 	(wire
 		(pts
-			(xy 125.73 71.12) (xy 127 71.12)
-		)
-		(stroke
-			(width 0)
-			(type default)
-		)
-	)
-	(wire
-		(pts
 			(xy 107.95 143.51) (xy 114.3 143.51)
 		)
@@
 	(wire
 		(pts
+			(xy 125.73 73.66) (xy 125.73 77.47)
+		)
+		(stroke
+			(width 0)
+			(type default)
+		)
+	)
+	(wire
+		(pts
 			(xy 62.23 34.29) (xy 62.23 41.91)
 		)
@@
 		)
 	)
-	(wire
-		(pts
-			(xy 123.19 67.31) (xy 123.19 77.47)
-		)
-		(stroke
-			(width 0)
-			(type default)
-		)
-	)
 	(polyline
 		(pts
@@
 	(wire
 		(pts
+			(xy 123.19 77.47) (xy 123.19 74.93)
+		)
+		(stroke
+			(width 0)
+			(type default)
+		)
+	)
+	(wire
+		(pts
 			(xy 66.802 135.89) (xy 74.422 135.89)
 		)
@@
 		)
 	)
+	(wire
+		(pts
+			(xy 123.19 74.93) (xy 118.11 74.93)
+		)
+		(stroke
+			(width 0)
+			(type default)
+		)
+	)
 	(polyline
 		(pts
@@
 		)
 	)
-	(wire
-		(pts
-			(xy 63.5 85.09) (xy 76.2 85.09)
-		)
-		(stroke
-			(width 0)
-			(type default)
-		)
-	)
 	(polyline
 		(pts
@@
 		)
 	)
-	(wire
-		(pts
-			(xy 125.73 71.12) (xy 125.73 77.47)
-		)
-		(stroke
-			(width 0)
-			(type default)
-		)
-	)
 	(polyline
 		(pts
@@
 		)
 	)
-	(label "IO15"
-		(at 63.5 85.09 0)
-		(effects
-			(font
-				(size 1.27 1.27)
-			)
-			(justify left bottom)
-		)
-	)
 	(label "ESP_MISO"
 		(at 125.73 44.45 180)
@@
 	(symbol
 		(lib_id "power:GND")
-		(at 127 71.12 90)
-		(unit 1)
-		(body_style 1)
-		(exclude_from_sim no)
-		(in_bom yes)
-		(on_board yes)
-		(in_pos_files yes)
-		(dnp no)
-		(property "Reference" "#PWR026"
-			(at 133.35 71.12 0)
-			(hide yes)
-			(show_name no)
-			(do_not_autoplace no)
-			(effects
-				(font
-					(size 1.27 1.27)
-				)
-			)
-		)
-		(property "Value" "GND"
-			(at 134.112 71.12 90)
-			(show_name no)
-			(do_not_autoplace no)
-			(effects
-				(font
-					(size 1.27 1.27)
-				)
-				(justify left)
-			)
-		)
-		(property "Footprint" ""
-			(at 127 71.12 0)
-			(hide yes)
-			(show_name no)
-			(do_not_autoplace no)
-			(effects
-				(font
-					(size 1.27 1.27)
-				)
-			)
-		)
-		(property "Datasheet" ""
-			(at 127 71.12 0)
-			(hide yes)
-			(show_name no)
-			(do_not_autoplace no)
-			(effects
-				(font
-					(size 1.27 1.27)
-				)
-			)
-		)
-		(property "Description" "Power symbol creates a global label with name \"GND\" , ground"
-			(at 127 71.12 0)
-			(hide yes)
-			(show_name no)
-			(do_not_autoplace no)
-			(effects
-				(font
-					(size 1.27 1.27)
-				)
-			)
-		)
-		(pin "1"
-		)
-		(instances
-			(project "DarkMagic"
-				(path "/8bdb7bb0-7fad-47bb-9a1b-904625b99d57"
-					(reference "#PWR026")
-					(unit 1)
-				)
-			)
-		)
-	)
-	(symbol
-		(lib_id "power:GND")
 		(at 72.39 120.65 270)
 		(unit 1)
@@
 	(symbol
 		(lib_id "power:+3V3")
-		(at 123.19 67.31 0)
+		(at 125.73 73.66 0)
 		(unit 1)
 		(body_style 1)
@@
 		(dnp no)
 		(property "Reference" "#PWR014"
-			(at 123.19 71.12 0)
+			(at 125.73 77.47 0)
 			(hide yes)
 			(show_name no)
@@
 		)
 		(property "Value" "+3V3"
-			(at 120.65 63.246 0)
+			(at 123.19 69.596 0)
 			(show_name no)
 			(do_not_autoplace no)
@@
 		)
 		(property "Footprint" ""
-			(at 123.19 67.31 0)
+			(at 125.73 73.66 0)
 			(hide yes)
 			(show_name no)
@@
 		)
 		(property "Datasheet" ""
-			(at 123.19 67.31 0)
+			(at 125.73 73.66 0)
 			(hide yes)
 			(show_name no)
@@
 		)
 		(property "Description" "Power symbol creates a global label with name \"+3V3\""
-			(at 123.19 67.31 0)
+			(at 125.73 73.66 0)
 			(hide yes)
 			(show_name no)
