File: PCB/fan_controller.kicad_sch (KiCad schematic)
At the start: 26 parts, among them IC17 LM393DR, J7 171825-2, M1 FFB0412VHN-B, Q2 SQ2348ES-T1_BE3

Commit message: KiCad: adjust PCB coords, routing & schematic
Minor PCB and schematic tweaks: update resistor and via Y coordinates in DarkMagic.kicad_pcb, adjust F.Cu routing segments (added one segment, changed segment endpoints and UUIDs) to clean up trace geometry, and change active_layer from 2 to 5 in DarkMagic.kicad_prl. Also correct schematic text in fan_controller.kicad_sch (LM3460 -> LMR33640) to fix part reference/notes.
Other:
- note added: "Fan Controller Set to turn on a fan when temperatures reach ~65° C. Thermistors measure the temperature of the LMR33640 and the AP63205. LM393DR follows OR Logic. Incorporates a ~0.5 second soft-start. C41 is an ALUMINUM capacitor!"
- note removed: "Fan Controller Set to turn on a fan when temperatures reach ~65° C. Thermistors measure the temperature of the LM3460 and the AP63205. LM393DR follows OR Logic. Incorporates a ~0.5 second soft-start. C41 is an ALUMINUM capacitor!"
Changed lines of the file:
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@@
 		)
 	)
-	(text "Fan Controller\n\nSet to turn on a fan when temperatures reach ~65° C.\n\nThermistors measure the temperature of the LM3460 \nand the AP63205. LM393DR follows OR Logic.\n\nIncorporates a ~0.5 second soft-start.\n\nC41 is an ALUMINUM capacitor!"
+	(text "Fan Controller\n\nSet to turn on a fan when temperatures reach ~65° C.\n\nThermistors measure the temperature of the LMR33640 \nand the AP63205. LM393DR follows OR Logic.\n\nIncorporates a ~0.5 second soft-start.\n\nC41 is an ALUMINUM capacitor!"
 		(exclude_from_sim no)
 		(at 166.116 29.972 0)
